Commit message: add pal_gripper camera

File: pal_gripper_description/urdf/cam_gripper.urdf.xacro (robot description, xacro)
@@ -53,4 +53,44 @@
     <axis xyz="0 0 0" />
   </joint>
+<!-- Camera -->
+    <joint name="camera_joint" type="fixed">
+      <origin xyz="0.065 0 -0.08" rpy="0 ${pi/2} ${pi}"/>
+      <parent link="${name}_link"/>
+      <child link="camera_link"/>
+      <axis xyz="0 0 0" />
+    </joint>
+    <link name="camera_link">
+      <collision>
+        <origin xyz="0 0 0" rpy="0 0 0"/>
+        <geometry>
+        <box size="0.05 0.01 0.01"/>
+        </geometry>
+      </collision>
+      <visual>
+        <origin xyz="0 0 0" rpy="0 0 0"/>
+        <geometry>
+        <box size="0.05 0.01 0.01"/>
+        </geometry>
+        <material name="Black"/>
+      </visual>
+      <inertial>
+        <mass value="1e-5" />
+        <origin xyz="0 0 0" rpy="0 0 0"/>
+        <inertia ixx="1e-6" ixy="0" ixz="0" iyy="1e-6" iyz="0" izz="1e-6" />
+      </inertial>
+    </link> <!---->
+    <!-- generate an optical frame http://www.ros.org/reps/rep-0103.html#suffix-frames
+        so that ros and opencv can operate on the camera frame correctly
+        these values have to be these values otherwise the gazebo camera image
+          won't be aligned properly with the frame it is supposedly originating from-->
+    <!-- -->
+    <joint name="camera_optical_joint" type="fixed">
+      <origin xyz="0 0 0" rpy="${-pi/2} 0 ${-pi/2}"/>
+      <parent link="camera_link"/>
+      <child link="camera_link_optical"/>
+    </joint>
+    <link name="camera_link_optical">
+    </link>
+   <!-- -->
   <link name="${name}_right_finger_link">
     <inertial>
@@ -148,44 +188,4 @@
   <xacro:finger_gazebo name="${name}_left_finger"/>
   <xacro:finger_gazebo name="${name}_right_finger"/>
-  <!-- Camera -->
-    <joint name="camera_joint" type="fixed">
-      <origin xyz="0 0.045 -0.08" rpy="0 ${pi/2} ${pi/2}"/>
-      <parent link="${name}_link"/>
-      <child link="camera_link"/>
-      <axis xyz="0 0 0" />
-    </joint>
-    <link name="camera_link">
-      <collision>
-        <origin xyz="0 0 0" rpy="0 0 0"/>
-        <geometry>
-        <box size="0.05 0.01 0.01"/>
-        </geometry>
-      </collision>
-      <visual>
-        <origin xyz="0 0 0" rpy="0 0 0"/>
-        <geometry>
-        <box size="0.05 0.01 0.01"/>
-        </geometry>
-        <material name="Black"/>
-      </visual>
-      <inertial>
-        <mass value="1e-5" />
-        <origin xyz="0 0 0" rpy="0 0 0"/>
-        <inertia ixx="1e-6" ixy="0" ixz="0" iyy="1e-6" iyz="0" izz="1e-6" />
-      </inertial>
-    </link> <!---->
-    <!-- generate an optical frame http://www.ros.org/reps/rep-0103.html#suffix-frames
-        so that ros and opencv can operate on the camera frame correctly
-        these values have to be these values otherwise the gazebo camera image
-          won't be aligned properly with the frame it is supposedly originating from-->
-    <!-- -->
-    <joint name="camera_optical_joint" type="fixed">
-      <origin xyz="0 0 0" rpy="${-pi/2} 0 ${-pi/2}"/>
-      <parent link="camera_link"/>
-      <child link="camera_link_optical"/>
-    </joint>
-    <link name="camera_link_optical">
-    </link>
-   <!-- -->
  </xacro:macro>
 </robot>

File: pal_gripper_description/urdf/gripper.gazebo.xacro (robot description, xacro)
@@ -24,3 +24,42 @@
     </gazebo>
   </xacro:macro>
+  <gazebo reference="camera_link">
+    <sensor name="camera1" type="camera">
+      <update_rate>30.0</update_rate>
+      <camera name="cam_gripper">
+        <horizontal_fov>1.3962634</horizontal_fov>
+        <image>
+          <width>800</width>
+          <height>800</height>
+          <format>R8G8B8</format>
+        </image>
+        <clip>
+          <near>0.02</near>
+          <far>300</far>
+        </clip>
+        <noise>
+          <type>gaussian</type>
+          <!-- Noise is sampled independently per pixel on each frame.
+               That pixel's noise value is added to each of its color
+               channels, which at that point lie in the range [0,1]. -->
+          <mean>0.0</mean>
+          <stddev>0.007</stddev>
+        </noise>
+      </camera>
+      <plugin filename="libgazebo_ros_camera.so" name="camera_controller">
+        <alwaysOn>true</alwaysOn>
+        <updateRate>0.0</updateRate>
+        <cameraName>camera1</cameraName>
+        <imageTopicName>image_raw</imageTopicName>
+        <cameraInfoTopicName>camera_info</cameraInfoTopicName>
+        <frameName>camera_link</frameName>
+        <hackBaseline>0.07</hackBaseline>
+        <distortionK1>0.0</distortionK1>
+        <distortionK2>0.0</distortionK2>
+        <distortionK3>0.0</distortionK3>
+        <distortionT1>0.0</distortionT1>
+        <distortionT2>0.0</distortionT2>
+      </plugin>
+    </sensor>
+  </gazebo>
 </robot>
